File: 20689/20689.sch (KiCad schematic (older format))
At the start: 1 part

Commit message: Hope for the best
Parts:
- U?: symbol ICM-20689:ICM-20689 -> 20689-rescue:ICM-20689-ICM-20689
Changed lines of the file:
@@
 EESchema Schematic File Version 4
+LIBS:20689-cache
 EELAYER 29 0
 EELAYER END
@@
 $EndDescr
 $Comp
-L ICM-20689:ICM-20689 U?
+L 20689-rescue:ICM-20689-ICM-20689 U?
 U 1 1 5D41AFC9
 P 4500 3750
