File: BMI088/BMI088.sch (KiCad schematic (older format))
At the start: 1 part

Commit message: Hole for the best 2
Parts:
- U?: symbol BMI088:BMI088 -> BMI088-rescue:BMI088-BMI088
Changed lines of the file:
@@
 EESchema Schematic File Version 4
+LIBS:BMI088-cache
 EELAYER 29 0
 EELAYER END
@@
 $EndDescr
 $Comp
-L BMI088:BMI088 U?
+L BMI088-rescue:BMI088-BMI088 U?
 U 1 1 5D4B6DE1
 P 5550 4050
