File: Development/Flight_Controller.sch (KiCad schematic (older format))
At the start: 22 parts, among them U1 STM32F765IIT6

Commit message: Begun labelling connectors with pinout document
Parts:
- removed C? (x8): Conn_6_1, symbol flightController:Conn_6_1
- removed C? (x4): Conn_4_1, symbol flightController:Conn_4_1
- removed C? (x2): Conn_5_1, symbol flightController:Conn_5_1
- removed C?: Conn_8_1, symbol flightController:Conn_8_1
- removed C? (x2): Conn_3_1, symbol flightController:Conn_3_1
- removed C? (x3): Conn_10_1, symbol flightController:Conn_10_1
- removed C?: Conn_7_1, symbol flightController:Conn_7_1
- removed U1: STM32F765IIT6, Package_QFP:LQFP-176_24x24mm_P0.5mm, symbol MCU_ST_STM32F7:STM32F765IITx
- added C? (x8): Conn_6_1, symbol flightController:Conn_6_1
- added C? (x4): Conn_4_1, symbol flightController:Conn_4_1
- added C?: Conn_5_1, symbol flightController:Conn_5_1
- added C?: Conn_8_1, symbol flightController:Conn_8_1
- added C? (x2): Conn_3_1, symbol flightController:Conn_3_1
- added C? (x3): Conn_10_1, symbol flightController:Conn_10_1
- added C?: Conn_7_1, symbol flightController:Conn_7_1
- added U?: STM32F765IIT6, Package_QFP:LQFP-176_24x24mm_P0.5mm, symbol MCU_ST_STM32F7:STM32F765IITx
Connections:
- wire segments 179 -> 182
Other:
- note added: "DSM/SBUS RC"
- note removed: "DSM RC"
- note removed: "SBUS RC"

Commit message: Updated Wiring
- 3 Sensors connected, some might need to change. Definitely needs to be double-checked at some point.
- All labels are now global
Parts:
- removed C? (x2): Conn_6_1, symbol flightController:Conn_6_1
- added C? (x4): 100nF, symbol Device:C
- added C? (x6): 47uF, symbol Device:C
- added C?: 4.7uF, symbol Device:C_Small
- added C? (x3): 100nF, symbol Device:C_Small
- added C?: 470nF, symbol Device:C_Small
- added D?: 1N5822, Diode_THT:D_DO-201AD_P15.24mm_Horizontal, symbol Diode:1N5822
- added J?: POWER1, symbol Connector_Generic:Conn_01x06
- added J?: POWER2, symbol Connector_Generic:Conn_01x06
- added R? (x2): 0R, symbol Device:R
- added R? (x2): 1K, symbol Device:R
- added R? (x2): 10K, symbol Device:R
- added R?: 220R, symbol Device:R
- added U? (x2): MIC5330-SSYML, symbol Flight_Controller-rescue:MIC5330-SSYML-FlightController-PowerSupply-rescue
- added U?: MIC5330-SPYML, symbol Flight_Controller-rescue:MIC5330-SPYML-FlightController-PowerSupply-rescue
- added U?: BMI088, symbol Symbol_Library:BMI088
- added U?: DPS422, symbol Symbol_Library:DPS422
- added U?: ICM20689, symbol Symbol_Library:ICM20689
- added U?: IST8310, symbol Symbol_Library:IST8310
- C? (x6): symbol flightController:Conn_6_1 -> Flight_Controller-rescue:Conn_6_1-flightController
- C? (x4): symbol flightController:Conn_4_1 -> Flight_Controller-rescue:Conn_4_1-flightController
- C?: symbol flightController:Conn_5_1 -> Flight_Controller-rescue:Conn_5_1-flightController
- C?: symbol flightController:Conn_8_1 -> Flight_Controller-rescue:Conn_8_1-flightController
- C? (x2): symbol flightController:Conn_3_1 -> Flight_Controller-rescue:Conn_3_1-flightController
- C? (x3): symbol flightController:Conn_10_1 -> Flight_Controller-rescue:Conn_10_1-flightController
- C?: symbol flightController:Conn_7_1 -> Flight_Controller-rescue:Conn_7_1-flightController
Connections:
- net labels added: D2_3V3, IMU_3V3, IMU_IO_3V3, IMU_VDD_3V0, IO1_3V3, MAIN_BAT1_I, MAIN_BAT1_V, MCU_3V3, SD_3V3, VBAT, VDD_SUP_IN, VREF+, VREF-, VSSA
- wire segments 182 -> 278
- no-connect marks 0 -> 19
Other:
- note removed: "POWER1"
- note removed: "POWER2"
- moved on the sheet: U?

Commit message: Crystal oscillator circuit added
Parts:
- added C? (x2): 8pF, symbol Device:C
- added Y?: NX3225SA, symbol Device:Crystal_GND24
- U?: symbol Symbol_Library:BMI088 -> Flight_Controller-rescue:BMI088-Symbol_Library
- U?: symbol Symbol_Library:DPS422 -> Flight_Controller-rescue:DPS422-Symbol_Library
- U?: symbol Symbol_Library:ICM20689 -> Flight_Controller-rescue:ICM20689-Symbol_Library
- U?: symbol Symbol_Library:IST8310 -> Flight_Controller-rescue:IST8310-Symbol_Library
Connections:
- wire segments 278 -> 296
Other:
- note added: "On-board sensors"
- note added: "Ports"
- note added: "Power management"
- moved on the sheet: C?

Commit message: wiring updates
Parts:
- removed C? (x6): 47uF, symbol Device:C
- added C? (x6): 47uF, symbol Device:C
Connections:
- wire segments 296 -> 304
Other:
- moved on the sheet: C?, D?, J?, R?, U?

Commit message: Updated power connections
All power components have been connected to the appropriate places
Parts:
- removed R?: 0R, symbol Device:R
- added C? (x9): 100nF, symbol Device:C
- added C? (x2): 2.2uF, symbol Device:C
- added R? (x2): 0R, symbol Device:R
- added R? (x3): 10K, symbol Device:R
- added U?: EG5350CT, symbol FlightController:EG5350CT
Connections:
- net labels added: BOOT0, VDDA
- net labels removed: VREF-
- wire segments 304 -> 364
Other:
- moved on the sheet: C?, R?

Commit message: Organised layout of schematic
Parts:
- U?: symbol FlightController:EG5350CT -> Flight_Controller-rescue:EG5350CT-FlightController
Other:
- moved on the sheet: C?, D?, J?, R?, U?, Y?

Commit message: Minor changes
Other:
- moved on the sheet: C?, U?

Commit message: Sensor & FRAM Update
Parts:
- added C? (x2): 100nF, symbol Device:C_Small
- added C? (x2): 2.2uF, symbol Device:C_Small
- added C?: 0.1uF, symbol Device:C_Small
- added C?: 220nF, symbol Device:C_Small
- added L?: L, symbol Device:L
- added R? (x3): 1K, symbol Device:R
- added R?: 10K, symbol Device:R
- added U?: FM25V02-G, symbol flightController:FM25V02-G
Connections:
- net GND: now also U?.2 (NC), C?.1, C?.1, C?.1, C?.1, C?.2, C?.2, R?.1, R?.2, U?.4 (GND)
- net IMU_3V3: now also L?.1, R?.2
- net IMU_VDD_3V0: now also C?.2, C?.2, C?.2
- net MCU_3V3: now also R?.1, U?.8 (3V3)
- net SPI1_CS1_ICM20689: now also R?.2
- net SPI2_CS_FRAM: now also U?.1 (CS)
- net SPI2_MISO_FRAM: now also U?.2 (MISO)
- net SPI2_MOSI_FRAM: now also U?.5 (MOSI)
- net SPI2_SCK_FRAM: now also U?.6 (SCK)
- net COM_VCC: now reaches U?.13 (DVDD)
- net COM_VCC: now also U?.2 (AVDD), C?.1, C?.1, L?.2
- net at U?.14 (RSTN): now also C?.2
- net at U?.5 (CAD0): now also R?.1
- net at U?.6 (CAD1): now also R?.1
- no-connect marks 19 -> 18
Other:
- note added: "FRAM"
- note added: "Just double check this symbol aligns with the \nFM25V02 and not just the FM25V01.\n"
