File: Development/Flight_Controller.sch (KiCad schematic (older format))
At the start: 95 parts, among them J1 POWER1, J2 POWER2, U1 ICM20689, U10 STM32F765IIT6, U2 MIC5330-SSYML, U3 MIC5330-SSYML, U4 MIC5330-SPYML, U5 MS5611-01BA, U6 BMI088, U7 IST8310, U8 TL3305AF160QG, U9 FM25V02-G, Y1 NX3225SA-24.000M-STD-CSR-1

Commit message: Updated schematics, added USB-C Port, etc.
Parts:
- removed C34: Conn_4_1, symbol Flight_Controller-rescue:Conn_4_1-flightController
- removed Y1: NX3225SA-24.000M-STD-CSR-1, SamacSys_Parts:NX3225SA12000MHZSTDCSR1, symbol SamacSys_Parts:NX3225SA-24.000M-STD-CSR-3
- added C?: 47uF, symbol Device:C
- added C?: 100nF, symbol Device:C
- added J?: USB_C_Receptacle, Connector_USB:USB_C_Receptacle_Amphenol_12401610E4-2A_CircularHoles, symbol Connector:USB_C_Receptacle
- added R?: 10K, symbol Device:R
- added R?: 50K, symbol Device:R
- added U?: TPS3808, symbol Flight_Controller-rescue:TPS3808
- added Y?: Crystal, symbol Device:Crystal
- C?: renamed from C7; footprint Capacitors_SMD:C_0603_HandSoldering -> (none)
- C?: renamed from C35; footprint Capacitors_SMD:C_0603_HandSoldering -> (none)
- C?: renamed from C9; footprint Capacitors_SMD:C_0603_HandSoldering -> (none)
- C?: renamed from C8; footprint Capacitors_SMD:C_0603_HandSoldering -> (none)
- C?: renamed from C42; footprint Capacitors_SMD:C_0603_HandSoldering -> (none)
- C?: renamed from C43; value 8pF -> 27pF; footprint Capacitors_SMD:C_0603_HandSoldering -> (none)
- C?: renamed from C20; footprint Capacitors_SMD:C_0603_HandSoldering -> (none)
- C?: renamed from C23; footprint Capacitors_SMD:C_0603_HandSoldering -> (none)
- C?: renamed from C21; footprint Capacitors_SMD:C_0603_HandSoldering -> (none)
- C?: renamed from C24; footprint Capacitors_SMD:C_0603_HandSoldering -> (none)
- C?: renamed from C25; footprint Capacitors_SMD:C_0603_HandSoldering -> (none)
- C?: renamed from C22; footprint Capacitors_SMD:C_0603_HandSoldering -> (none)
- C?: renamed from C36; footprint Capacitors_SMD:C_0603_HandSoldering -> (none)
- C?: renamed from C32; footprint Capacitors_SMD:C_0603_HandSoldering -> (none)
- C?: renamed from C38; footprint Capacitors_SMD:C_0603_HandSoldering -> (none)
- C?: renamed from C1; footprint Capacitors_SMD:C_0603_HandSoldering -> (none)
- C?: renamed from C52; footprint Capacitors_SMD:C_0603_HandSoldering -> (none)
- C?: renamed from C53; footprint Capacitors_SMD:C_0603_HandSoldering -> (none)
- C?: renamed from C47; footprint Capacitors_SMD:C_0603_HandSoldering -> (none)
- C?: renamed from C46; footprint Capacitors_SMD:C_0603_HandSoldering -> (none)
- C?: renamed from C45; footprint Capacitors_SMD:C_0603_HandSoldering -> (none)
- C?: renamed from C44; footprint Capacitors_SMD:C_0603_HandSoldering -> (none)
- C?: renamed from C31; footprint Capacitors_SMD:C_0603_HandSoldering -> (none)
- C?: renamed from C48; footprint Capacitors_SMD:C_0603_HandSoldering -> (none)
- C?: renamed from C49; footprint Capacitors_SMD:C_0603_HandSoldering -> (none)
- C?: renamed from C50; footprint Capacitors_SMD:C_0603_HandSoldering -> (none)
- C?: renamed from C39; footprint Capacitors_SMD:C_0603_HandSoldering -> (none)
- C?: renamed from C37; footprint Capacitors_SMD:C_0603_HandSoldering -> (none)
- C?: renamed from C10; footprint Capacitors_SMD:C_0603_HandSoldering -> (none)
- C?: renamed from C11; footprint Capacitors_SMD:C_0603_HandSoldering -> (none)
- C?: renamed from C51; footprint Capacitors_SMD:C_0603_HandSoldering -> (none)
- C?: renamed from C40; footprint Capacitors_SMD:C_0603_HandSoldering -> (none)
- C?: renamed from C26; footprint Capacitors_SMD:C_0603_HandSoldering -> (none)
- C?: renamed from C27; footprint Capacitors_SMD:C_0603_HandSoldering -> (none)
- C?: renamed from C28; footprint Capacitors_SMD:C_0603_HandSoldering -> (none)
- D?: renamed from D1; footprint (none) -> Diode_THT:D_DO-201AD_P15.24mm_Horizontal
- R?: renamed from R5; footprint Resistors_SMD:R_0603_HandSoldering -> (none)
- R?: renamed from R12; footprint Resistors_SMD:R_0603_HandSoldering -> (none)
- R?: renamed from R8; footprint Resistors_SMD:R_0603_HandSoldering -> (none)
- R?: renamed from R4; footprint Resistors_SMD:R_0603_HandSoldering -> (none)
- R?: renamed from R2; footprint Resistors_SMD:R_0603_HandSoldering -> (none)
- R?: renamed from R6; footprint Resistors_SMD:R_0603_HandSoldering -> (none)
- R?: renamed from R3; footprint Resistors_SMD:R_0603_HandSoldering -> (none)
- R?: renamed from R10; footprint Resistors_SMD:R_0603_HandSoldering -> (none)
- R?: renamed from R11; footprint Resistors_SMD:R_0603_HandSoldering -> (none)
- R?: renamed from R7; footprint Resistors_SMD:R_0603_HandSoldering -> (none)
- R?: renamed from R23; footprint Resistors_SMD:R_0603_HandSoldering -> (none)
- R?: renamed from R16; footprint Resistors_SMD:R_0603_HandSoldering -> (none)
- R?: renamed from R15; footprint Resistors_SMD:R_0603_HandSoldering -> (none)
- R?: renamed from R9; footprint Resistors_SMD:R_0603_HandSoldering -> (none)
- R?: renamed from R13; footprint Resistors_SMD:R_0603_HandSoldering -> (none)
- R?: renamed from R22; footprint Resistors_SMD:R_0603_HandSoldering -> (none)
- R?: renamed from R19; footprint Resistors_SMD:R_0603_HandSoldering -> (none)
- R?: renamed from R20; footprint Resistors_SMD:R_0603_HandSoldering -> (none)
- R?: renamed from R1; footprint Resistors_SMD:R_0603_HandSoldering -> (none)
- R?: renamed from R14; footprint Resistors_SMD:R_0603_HandSoldering -> (none)
- R?: renamed from R24; footprint Resistors_SMD:R_0603_HandSoldering -> (none)
- R?: renamed from R26; footprint Resistors_SMD:R_0603_HandSoldering -> (none)
- R?: renamed from R25; footprint Resistors_SMD:R_0603_HandSoldering -> (none)
- R?: renamed from R27; footprint Resistors_SMD:R_0603_HandSoldering -> (none)
- R?: renamed from R17; footprint Resistors_SMD:R_0603_HandSoldering -> (none)
- R?: renamed from R18; footprint Resistors_SMD:R_0603_HandSoldering -> (none)
- R?: renamed from R21; footprint Resistors_SMD:R_0603_HandSoldering -> (none)
- U?: renamed from U2; footprint MIC5330-SSYML-TR:MIC5330-SSYML-TR -> (none)
- U?: renamed from U4; footprint MIC5330-SSYML-TR:MIC5330-SSYML-TR -> (none)
- U?: renamed from U3; footprint MIC5330-SSYML-TR:MIC5330-SSYML-TR -> (none)
- U?: renamed from U8; value TL3305AF160QG -> EG5350CT; footprint SamacSys_Parts:TL3305AF160QG -> (none)
- renumbered C30 to C?, C2 to C?, C12 to C?, C13 to C?, C19 to C?, C3 to C?, C17 to C?, C4 to C?, C16 to C?, C18 to C?, C15 to C?, C5 to C?, C41 to C?, C6 to C?, C33 to C?, C29 to C?, C14 to C?, J1 to J?, J2 to J?, L1 to L?, U10 to U?, U6 to U?, U1 to U?, U5 to U?, U7 to U?, U9 to U?
Connections:
- net labels added: FMU_RESET, NRST, OTG_N, OTG_P, USB_VCC
- wire segments 445 -> 466
- no-connect marks 28 -> 40
Other:
- note removed: "USB"
- moved on the sheet: C?, R?, U?

Commit message: Stability update, ensuring all files are up to date
Parts:
- U? (x3): footprint (none) -> FLIGHTFOOT:MIC5330-SSYML-TR
- U?: footprint (none) -> FLIGHTFOOT:BMI088
- U?: footprint (none) -> FLIGHTFOOT:ICM20689
- U?: footprint (none) -> FLIGHTFOOT:ms5611
- U?: footprint (none) -> FLIGHTFOOT:ist8310
- U?: footprint (none) -> FLIGHTFOOT:FM25V02-G
Other:
- note removed: "Need to double check"
Changed lines of the file:
@@
 F 0 "U?" H 2800 2975 50  0000 C CNN
 F 1 "MIC5330-SSYML" H 2500 2225 50  0000 C CNN
-F 2 "" H 2450 2975 50  0001 C CNN
+F 2 "FLIGHTFOOT:MIC5330-SSYML-TR" H 2450 2975 50  0001 C CNN
 F 3 "" H 2450 2975 50  0001 C CNN
 	1    2500 2625
@@
 F 0 "U?" H 2800 5325 50  0000 C CNN
 F 1 "MIC5330-SPYML" H 2500 4575 50  0000 C CNN
-F 2 "" H 2450 5325 50  0001 C CNN
+F 2 "FLIGHTFOOT:MIC5330-SSYML-TR" H 2450 5325 50  0001 C CNN
 F 3 "" H 2450 5325 50  0001 C CNN
 	1    2500 4975
@@
 F 0 "U?" H 2800 4175 50  0000 C CNN
 F 1 "MIC5330-SSYML" H 2500 3425 50  0000 C CNN
-F 2 "" H 2450 4175 50  0001 C CNN
+F 2 "FLIGHTFOOT:MIC5330-SSYML-TR" H 2450 4175 50  0001 C CNN
 F 3 "" H 2450 4175 50  0001 C CNN
 	1    2500 3825
@@
 F 0 "U?" H 6100 10265 50  0000 C CNN
 F 1 "BMI088" H 6100 10174 50  0000 C CNN
-F 2 "" H 6100 9500 50  0001 C CNN
+F 2 "FLIGHTFOOT:BMI088" H 6100 9500 50  0001 C CNN
 F 3 "" H 6100 9500 50  0001 C CNN
 	1    6100 9500
@@
 F 0 "U?" H 3144 12021 50  0000 L CNN
 F 1 "ICM20689" H 3144 11930 50  0000 L CNN
-F 2 "" H 2900 12550 50  0001 C CNN
+F 2 "FLIGHTFOOT:ICM20689" H 2900 12550 50  0001 C CNN
 F 3 "" H 2900 12550 50  0001 C CNN
 	1    2450 12000
@@
 F 0 "U?" H 6325 12115 50  0000 C CNN
 F 1 "IST8310" H 6325 12024 50  0000 C CNN
-F 2 "" H 6950 12150 50  0001 C CNN
+F 2 "FLIGHTFOOT:ist8310" H 6950 12150 50  0001 C CNN
 F 3 "" H 6950 12150 50  0001 C CNN
 	1    6250 11750
@@
 F 0 "U?" H 13450 2875 50  0000 C CNN
 F 1 "FM25V02-G" H 13450 2784 50  0000 C CNN
-F 2 "" H 13450 3100 50  0001 C CNN
+F 2 "FLIGHTFOOT:FM25V02-G" H 13450 3100 50  0001 C CNN
 F 3 "" H 13450 3100 50  0001 C CNN
 	1    13450 2450
@@
 F 0 "U?" H 2775 9675 50  0000 C CNN
 F 1 "MS5611-01BA" H 2775 9584 50  0000 C CNN
-F 2 "" H 2150 9700 50  0001 C CNN
+F 2 "FLIGHTFOOT:ms5611" H 2150 9700 50  0001 C CNN
 F 3 "" H 2150 9700 50  0001 C CNN
 	1    2650 9200
@@
 Text Notes 17250 10100 3    50   ~ 0
 Not finished
-Text Notes 23450 15450 3    50   ~ 0
-Need to double check
-Text Notes 20750 4700 3    50   ~ 0
-Need to double check
 Text GLabel 3950 18800 2    50   Input ~ 0
 VDD_5V_IN

Commit message: Feature Update!
+ Data Translation, CAN Bus, I2C Rail, ADC Rail
+ SD Card ready to merge
+ New Formatting (Clean up)
Parts:
- added C43, C44, C45, C? (x8): 100nF, symbol Device:C_Small
- added C? (x4): 100nf, symbol Device:C
- added C? (x6): 47uF, symbol Device:C
- added C? (x3): 100nF, symbol Device:C
- added C?: Conn_4_1, symbol Flight_Controller-rescue:Conn_4_1-flightController
- added D?: D240L, symbol Device:D
- added LC1, LC2, LC3, LC? (x2): EMI_Filter_LC, symbol Device:EMI_Filter_C
- added R16, R17, R18, R19, R20, R21, R22, R23, R? (x12): 100, symbol Device:R
- added R25, R26: 10k, symbol Device:R
- added R28, R29: 120, symbol Device:R
- added R? (x12): 100R, symbol Device:R
- added R?: 1K, symbol Device:R
- added R? (x9): 10K, symbol Device:R
- added R? (x8): 1k5, symbol Device:R
- added R? (x4): 2M, symbol Device:R
- added U10: SN74LVC8T245, symbol Flight_Controller-rescue:SN74LVC8T245
- added U12, U13: TJA1051TK-3, Package_DFN_QFN:DFN-8-1EP_3x3mm_P0.65mm_EP1.55x2.4mm, symbol Interface_CAN_LIN:TJA1051TK-3
- added U? (x3): TXS0108EPW, Package_SO:TSSOP-20_4.4x6.5mm_P0.65mm, symbol Logic_LevelTranslator:TXS0108EPW
- added U?: NUF2042XV6T1G, symbol Flight_Controller-rescue:NUF2042XV6T1G
- gave numbers to parts that had none: 100
Connections:
- net IMU_IO_3V3 is gone; now on net IMU_3V3: C9.2, U1.8 (VDDIO)
- net VDD_SUP_IN is gone; now on net VCC: U4.1 (VIN)
- net ADC1_SPARE_1: now also C?.1, R?.1, R?.2
- net ADC1_SPARE_2: now also C?.1, R?.1, R?.2
- net BAT1_I: now also C?.2, R?.1
- net BAT1_V: now also C?.2, R?.1
- net BAT2_I: now also C?.2, R?.1
- net BAT2_V: now also C?.2, R?.1
- net CAN1_RX: now also U12.4 (RXD)
- net CAN1_TX: now also U12.1 (TXD)
- net CAN2_RX\(UART5_RX_ESC): now also U13.4 (RXD)
- net CAN2_TX\(UART5_TX_ESC): now also U13.1 (TXD)
- net FMU_CAP1: now also U?.9 (A8)
- net FMU_CAP2: now also U?.8 (A7)
- net FMU_CAP3: now also U?.7 (A6)
- net FMU_CH1: now also U10.10 (A8)
- net FMU_CH2: now also U10.9 (A7)
- net FMU_CH3: now also U10.8 (A6)
- net FMU_CH4: now also U10.7 (A5)
- net FMU_CH5: now also U10.6 (A4)
- net FMU_CH6: now also U10.5 (A3)
- net FMU_CH7: now also U10.4 (A2)
- net FMU_CH8: now also U10.3 (A1)
- net GND: now also C20.4, C30.4, C43.1, C43.2, C44.2, C45.2, C?.1, C?.1, C?.1, C?.1, C?.1, C?.1, C?.1, C?.1, C?.1, C?.1, C?.1, C?.1, C?.1, C?.1, C?.2, C?.2, C?.2, C?.2, C?.2, C?.2, C?.2, C?.2, C?.2, C?.4, LC1.3, LC2.3, LC3.3, LC?.3, LC?.3, R?.2, R?.2, R?.2, R?.2, R?.2, R?.2, R?.2, R?.2, U10.11 (GND), U10.12 (GND), U10.13 (GND), U10.22 (OE), U10.23 (VCCB), U10.24 (VCCB), U12.2 (GND), U12.9 (GND), U13.2 (GND), U13.9 (GND), U?.11 (GND), U?.11 (GND), U?.11 (GND), U?.19 (VCCB), U?.19 (VCCB), U?.2 (GND)
- net I2C1_SCL_GPS1: now also R?.1, R?.2; no longer C42.4
- net I2C1_SDA_GPS1: now also R?.1, R?.2; no longer C42.5
- net I2C2_SCL_UART4: now also R?.1, R?.2
- net I2C2_SDA_UART4: now also R?.1, R?.2
- net I2C3_SCL_EXTERNAL3: now also R?.1, R?.2
- net I2C3_SDA_EXTERNAL3: now also R?.1, R?.2
- net I2C4_SCL_EXTERNAL2: now also R?.1, R?.2
- net I2C4_SDA_EXTERNAL2: now also R?.1, R?.2
- net IMU_3V3: now also C?.2, R?.1
- net IMU_VDD_3V0: now also LC?.1; no longer C1.1, U5.1 (VDD)
- net IO1_3V3: now also C?.2, C?.2, C?.2, LC3.1, U10.1 (VCCA), U10.2 (DIR), U?.10 (OE), U?.10 (OE), U?.2 (VCCA), U?.2 (VCCA)
- net MCU_3V3: now also R25.1, R26.1, R?.2, R?.2, R?.2, R?.2, R?.2, R?.2, R?.2, R?.2, U12.5 (VIO), U13.5 (VIO)
- net OTG_N: now also U?.1 (D1_IN)
- net OTG_P: now also U?.3 (D2_IN)
- net SCALED_V5: now also C?.1, R?.1, R?.2
- net SCALED_VDD_3V3_SENSORS: now also C?.1, R?.1, R?.2
- net TF_3V3: now also C?.1
- net UART4_RX_I2C2: now also U?.7 (A6)
- net UART4_TX_I2C2: now also U?.6 (A5)
- net UART7_RX_DEBUG: now also U?.3 (A2)
- net UART7_TX_DEBUG: now also U?.1 (A1)
- net USART1_RX_GPS1: now also U?.4 (A3)
- net USART1_TX_GPS1: now also U?.5 (A4)
- net USART2_CTS_TELEM1: now also U?.5 (A4)
- net USART2_RTS_TELEM1: now also U?.4 (A3)
- net USART2_RX_TELEM1: now also U?.1 (A1)
- net USART2_TX_TELEM1: now also U?.3 (A2)
- net USART3_CTS_TELEM2: now also U?.8 (A7)
- net USART3_RTS_TELEM2: now also U?.9 (A8)
- net USART3_RX_TELEM2: now also U?.6 (A5)
- net USART3_TX_TELEM2: now also U?.7 (A6)
- net USB_VCC: now also D?.2 (A), R?.1, U?.5 (VBUS)
- net VBUS: now also R?.2
- net at C20.1: now also LC1.2
- net CAN_H_1: now reaches C20.2
- net CAN_H_1: now also R28.2, U12.7 (CANH)
- net CAN_L_1: now reaches C20.3
- net CAN_L_1: now also R28.1, U12.6 (CANL)
- net at C42.8: now also LC3.2
- net at C30.1: now also LC2.2
- net CAN_H_2: now reaches C30.2
- net CAN_H_2: now also R29.2, U13.7 (CANH)
- net CAN_L_2: now reaches C30.3
- net CAN_L_2: now also R29.1, U13.6 (CANL)
- net VDD_5V_IN renamed VCC
- net VCC: now also C44.1, C45.1, C?.1, C?.1, C?.2, C?.2, C?.2, C?.2, D?.1 (K), LC1.1, LC2.1, LC?.1, R?.1, R?.1, U12.3 (VCC), U13.3 (VCC); no longer U2.5 (EN1)
- net nARMED renamed TIM5_SPARE_4
- net TIM5_SPARE_4: now also U?.6 (A5)
- new net: R?.2, U2.5 (EN1)
- new net: C1.1, LC?.2, U5.1 (VDD)
- new net: R?.1, U?.14 (B6) (x2)
- new net: R?.1, U?.15 (B5) (x2)
- new net: R?.1, U?.16 (B4) (x2)
- new net: R?.1, U?.17 (B3) (x2)
- new net: R?.1, U?.12 (B8)
- new net: R?.1, U?.13 (B7)
- new net: R?.1, U?.18 (B2)
- new net: R?.1, U?.20 (B1)
- new net: R23.1, U10.14 (B8)
- new net: R22.1, U10.15 (B7)
- new net: R21.1, U10.16 (B6)
- new net: R20.1, U10.17 (B5)
- new net: R19.1, U10.18 (B4)
- new net: R18.1, U10.19 (B3)
- new net: R17.1, U10.20 (B2)
- new net: R16.1, U10.21 (B1)
- new net: C?.1, LC?.2
- new net ADC1_SPARE_1_CHANNEL: R?.1
- new net ADC1_SPARE_2_CHANNEL: R?.1
- new net CAN1_SILENT_S0: R25.2, U12.8 (S)
- new net CAN2_SILENT_S1: R26.2, U13.8 (S)
- new net GPS1_RX1: R?.2
- new net GPS1_TX1: R?.2
- new net I2C_2_SCL_PORT: R?.1
- new net I2C_2_SDA_PORT: R?.1
- new net I2C_3_SCL_PORT: R?.1
- new net I2C_3_SDA_PORT: R?.1
- new net I2C_4_SCL_PORT: C?.2, R?.1
- new net I2C_4_SDA_PORT: C?.3, R?.1
- new net OTG_FS_DM: U?.6 (D1_OUT)
- new net OTG_FS_DP: U?.4 (D2_OUT)
- new net OUT1: R23.2, R?.2
- new net OUT2: R22.2, R?.2
- new net OUT3: R21.2, R?.2
- new net OUT4: R20.2, R?.2
- new net OUT5: R19.2
- new net OUT6: R18.2
- new net OUT7: R17.2
- new net OUT8: R16.2
- new net SCL1_GPS: C42.4, R?.1
- new net SDA1_GPS: C42.5, R?.1
- new net UART4_RX: R?.2
- new net UART4_TX: R?.2
- new net UART7_RX: U?.18 (B2)
- new net UART7_TX: U?.20 (B1)
- new net USART2_CTS: R?.2
- new net USART2_RTS: R?.2
- new net USART2_RX: R?.2
- new net USART2_TX: R?.2
- new net USART3_CTS: R?.2
- new net USART3_RTS: R?.2
- new net USART3_RX: R?.2
- new net USART3_TX: R?.2
- no-connect marks 40 -> 52
Other:
- note added: "ADC RAIL"
- note added: "CAN BUS"
- note added: "DATA TRANSLATION"
- note added: "I2C RAIL"
- note added: "I2C4"
- note added: "ON-BOARD SENSORS"
- note added: "PORTS"
- note added: "POWER MANAGEMENT"
- note added: "VERSION"
- note removed: "On-board sensors"
- note removed: "Ports"
- note removed: "Power management"
- note removed: "missing LC EMI Filter Low Pass"
- moved on the sheet: C1, C10, C11, C12, C13, C14, C15, C16, C17, C18, C19, C2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

Commit message: Merged Status LED and SD Card
Parts:
- added C? (x2): 100nF, symbol Device:C
- added C? (x2): 100nf, symbol Device:C
- added C?: 47uF, symbol Device:C
- added D?: DIODE, symbol pspice:DIODE
- added D?: SMLVN6RGB, LED_SMD:LED_ROHM_SMLVN6, symbol LED:SMLVN6RGB
- added J?: Micro_SD_Card_Det, symbol Connector:Micro_SD_Card_Det
- added LC? (x4): EMI_Filter_LC, symbol Device:EMI_Filter_C
- added R? (x5): 10K, symbol Device:R
- added R? (x4): 10k, symbol pspice:R
- added R? (x2): 220R, symbol Device:R
- added R? (x2): 100, symbol Device:R
- added U?: SERVO_THING, symbol Flight_Controller-rescue:SERVO_THING
Connections:
- net GND: now also U?.19 (VCCB), C?.1, C?.1, C?.2, C?.2, C?.2, C?.2, J?.11 (SHIELD), J?.6 (VSS), LC?.3, LC?.3, LC?.3, R?.2, U?.~ (SERVO_VCC)
- net IO1_3V3: now also U?.10 (OE), U?.2 (VCCA), C?.2, LC?.1
- net OUT1: now also U?.2; no longer R?.2
- net OUT2: now also U?.3; no longer R?.2
- net OUT3: now also U?.4; no longer R?.2
- net OUT4: now also U?.5; no longer R?.2
- net OUT5: now also U?.6
- net OUT6: now also U?.7
- net OUT7: now also U?.8
- net OUT8: now also U?.9
- net RSSI_IN: now also R?.1
- net SDMMC1_CMD: now also J?.3 (CMD), R?.1
- net SDMMC1_D0: now also J?.7 (DAT0), R?.1
- net SDMMC1_D1: now also J?.8 (DAT1), R?.1
- net SDMMC1_D2: now also J?.1 (DAT2), R?.1
- net SDMMC1_D3: now also J?.2 (DAT3/CD), R?.1
- net TF_3V3: now also C?.1, C?.1, J?.4 (VDD), R?.2, R?.2, R?.2, R?.2, R?.2
- net VCC: now also C?.1, D?.1 (GA), D?.1 (K), D?.3 (RA), D?.5 (BA), LC?.1, LC?.2
- net nLED_BLUE: now also R?.2
- net nLED_GREEN: now also R?.2
- net nLED_RED: now also R?.2
- net at C14.1: now also LC?.1
- net at C14.2: now also R?.1
- net at C14.3: now also R?.2
- net at C14.4: now also LC?.2
- net at U?.12 (B8): now also R?.1
- net at U?.13 (B7): now also R?.1
- net at U?.14 (B6): now also R?.1
- net at U?.15 (B5): now also R?.1
- net USART6_TX_TELEM\(RC_INPUT) renamed USART6_TX_TELEM3\(RC_INPUT)
- net USART6_TX_TELEM3\(RC_INPUT): now also R?.2, R?.2
- new net: D?.2 (A), R?.1
- new net: D?.6 (BK), R?.1
- new net: D?.4 (RK), R?.1
- new net: D?.2 (GK), R?.1
- new net: LC?.2, U?.~ (SERVO_VCC)
- new net AUX1: R?.2, U?.10
- new net AUX2: R?.2, U?.11
- new net AUX3: R?.2, U?.12
- new net AUX4: R?.2, U?.13
- new net FMU_PPM_INPUT: R?.1, R?.2
- new net RC_IN_PORT: R?.1, U?.1
- new net SDIO1_CARD_DETECT: J?.10 (DET_A), J?.9 (DET_B)
- new net SDMMC1_CK: J?.5 (CLK)
- new net SERVO_VCC: U?.~ (SERVO_VCC)
Other:
- note added: "PWM I/O"
- note added: "SD CARD"
- note added: "STATUS LEDS"
- moved on the sheet: C1, C10, C11, C12, C13, C14, C15, C16, C17, C18, C19, C2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

Commit message: Finished Ports
Parts:
- removed LC?: EMI_Filter_LC, symbol Device:EMI_Filter_C
- added C? (x3): Conn_6_1, symbol Flight_Controller-rescue:Conn_6_1-flightController
- added C? (x3): Conn_4_1, symbol Flight_Controller-rescue:Conn_4_1-flightController
- added LC? (x6): EMI_Filter_LC, symbol Device:EMI_Filter_C
Connections:
- net ADC1_SPARE_1_CHANNEL: now also C?.2
- net ADC1_SPARE_2_CHANNEL: now also C?.3
- net GND: now also C2.6, C?.4, C?.4, C?.4, C?.6, C?.6, C?.6, LC?.3, LC?.3, LC?.3, LC?.3, LC?.3, LC?.3
- net GPS1_RX1: now also C42.3
- net GPS1_TX1: now also C42.2
- net I2C_2_SCL_PORT: now also C2.4
- net I2C_2_SDA_PORT: now also C2.5
- net I2C_3_SCL_PORT: now also C?.2, C?.2
- net I2C_3_SDA_PORT: now also C?.3, C?.3
- net UART4_RX: now also C2.3
- net UART4_TX: now also C2.2
- net UART7_RX: now also C?.3
- net UART7_TX: now also C?.2
- net USART1_RX_GPS1: no longer C42.3
- net USART1_TX_GPS1: no longer C42.2
- net USART2_CTS: now also C?.4
- net USART2_RTS: now also C?.5
- net USART2_RX: now also C?.3
- net USART2_TX: now also C?.2
- net USART3_CTS: now also C?.4
- net USART3_RTS: now also C?.5
- net USART3_RX: now also C?.3
- net USART3_TX: now also C?.2
- net VCC: now also C?.1, LC?.1, LC?.1, LC?.1, LC?.1, LC?.1, LC?.1; no longer C42.1
- net at C2.1: now also LC?.2
- new net: C42.1, LC?.2
- new net: C?.1, LC?.2 (x4)
- new net I2C2_VCC: C?.1
- new net JTAG_SWCLK: C?.5
- new net JTAG_SWDIO: C?.4
Other:
- note added: "ADC3/5"
- note added: "DSU7"
- note added: "I2C2"
- note added: "I2C3"
- note added: "OLD\nPORTS"
- note added: "UART4"
- note added: "USART2"
- note added: "USART3"
- note removed: "UART"
- moved on the sheet: C11, C12, C13, C14, C15, C16, C17, C18, C2, C20, C3, C30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

Commit message: Schematics 99% Finished
+ Double check capacitor values
+ Clarify VBAT connection
Parts:
- removed C11, C12, C17, C18, C3: Conn_6_1, symbol Flight_Controller-rescue:Conn_6_1-flightController
- removed C13, C4: Conn_3_1, symbol Flight_Controller-rescue:Conn_3_1-flightController
- removed C15: Conn_4_1, symbol Flight_Controller-rescue:Conn_4_1-flightController
- removed C16: Conn_8_1, symbol Flight_Controller-rescue:Conn_8_1-flightController
- removed C31, C40: Conn_10_1, symbol Flight_Controller-rescue:Conn_10_1-flightController
- added C? (x2): 12pF, symbol Device:C
- added LC?: EMI_Filter_LC, symbol Device:EMI_Filter_C
- added R?: 10K, symbol Device:R
- added R?: 0R, symbol Device:R
- added R?: 1M, symbol Device:R
- added Y?: Crystal, symbol Device:Crystal
- C46: value 8pF -> 27pF
Connections:
- net CAN3_SILENT_S0 is gone; now on net CAN1_SILENT_S0: U14.43 (PH2)
- net CAN3_SILENT_S1 is gone; now on net CAN2_SILENT_S1: U14.44 (PH3)
- net FMU_PPM_INPUT is gone; now on net RC_INPUT\(aka_PPM_IN): R?.1, R?.2
- net JTAG-SWCLK is gone; now on net JTAG_SWCLK: U14.137 (PA14)
- net JTAG-SWDIO is gone; now on net JTAG_SWDIO: U14.124 (PA13)
- net SDMMC1_CK is gone; now on net SDMMC1_CLK: J?.5 (CLK)
- net 16_MHZ_IN: now also C?.1, R?.2, Y?.1
- net 16_MHZ_OUT: now also C?.1, R?.1, Y?.2
- net GND: now also C?.2, C?.2, LC?.3, R?.1, R?.2; no longer U14.37 (VSSA)
- net SPI5_CS1_EXTERNAL1: now also C5.5
- net SPI5_CS2_EXTERNAL1: now also C5.6
- net SPI5_MISO_EXTERNAL1: now also C5.3
- net SPI5_MOSI_EXTERNAL1: now also C5.4
- net SPI5_SCK_EXTERNAL1: now also C5.2
- net VCC: now also LC?.1
- net 32KHz_OUT: now reaches C46.1, U14.10 (PC15), Y1.1
- net BOOT1: now reaches U14.58 (PB2)
- net BOOT1: now also R?.1
- net 32KHz_IN: now reaches C47.1, U14.9 (PC14), Y1.2
- net at C5.1: now also LC?.2
- new net: R?.2, U14.37 (VSSA)
- no-connect marks 52 -> 71
Other:
- note added: "SPI5"
- note removed: "CAP & ADC IN"
- note removed: "FMU DEBUG"
- note removed: "FMU PWM OUT"
- note removed: "I/O PWM OUT"
- note removed: "I2CA"
- note removed: "I2CB"
- note removed: "IO DEBUG"
- note removed: "Not finished"
- note removed: "OLD\nPORTS"
- note removed: "PPM RC"
- note removed: "SBUS OUT"
- note removed: "SPI"
- note removed: "TELEM1"
- note removed: "TELEM2"
- moved on the sheet: C5, J1

Commit message: Finished Schematics.
Parts:
- added BT?: Battery_Cell, symbol Device:Battery_Cell
Connections:
- net GND: now also BT?.2 (-); no longer C25.2, C43.2, C?.2, C?.2, C?.2, R4.2, U10.23 (VCCB), U10.24 (VCCB), U14.6 (VBAT), U3.7 (VOUT2), U?.19 (VCCB), U?.19 (VCCB), U?.19 (VCCB)
- new net D2_3V3: C25.2, C43.2, C?.2, C?.2, C?.2, U10.23 (VCCB), U10.24 (VCCB), U3.7 (VOUT2), U?.19 (VCCB), U?.19 (VCCB), U?.19 (VCCB)
- new net VBAT: BT?.1 (+), R4.2, U14.6 (VBAT)
Other:
- moved on the sheet: C46, C47, C48, C49, C50, C51, C52, C53, C54, C55, C56, C57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

Commit message: Error Fixing
Parts:
- removed C8: 100nF, symbol Device:C
- added C3: 100nF, symbol Device:C
- added LC10: EMI_Filter_LC, symbol Device:EMI_Filter_C
- gave numbers to parts that had none: 120
- renumbered C19 to C13, C27 to C15, C28 to C16, C29 to C17, C21 to C18, C22 to C19, C7 to C2, C23 to C20, C26 to C21, C24 to C22, C25 to C23, C32 to C26, C33 to C27, C36 to C28, C37 to C29, C38 to C30, C39 to C31, C34 to C32, C35 to C33, C41 to C34, C46 to C35, C47 to C36, C48 to C37, C49 to C38, C50 to C39, C6 to C4, C51 to C40, C52 to C41, C14 to C42, C42 to C43, C53 to C46, C54 to C47, C55 to C48, C56 to C49, C9 to C5, C57 to C50, C5 to C58, C20 to C59, C10 to C6, C30 to C60, C2 to C61, C44 to C74, C45 to C75, C43 to C76, J2 to J1, J3 to J2, J1 to J3, LC1 to LC14, LC2 to LC15, LC3 to LC4, R12 to R10, R24 to R103, R13 to R11, R14 to R12, R15 to R13, R27 to R14, R7 to R16, R10 to R17, R11 to R18, R30 to R22, R31 to R23, R32 to R24, R33 to R25, R34 to R26, R35 to R27, R36 to R29, R2 to R3, R37 to R30, R3 to R4, R16 to R48, R17 to R49, R4 to R5, R18 to R50, R19 to R51, R20 to R52, R21 to R53, R22 to R54, R23 to R55, R5 to R6, R6 to R7, R25 to R75, R26 to R76, R38 to R85, R39 to R86, R40 to R91, R41 to R92, R28 to R93, R29 to R94, U4 to U1, U14 to U10, U10 to U11, U11 to U15, U12 to U16, U13 to U17, U1 to U2, U2 to U4
Connections:
- net USB_DM is gone; now on net OTG_FS_DM: U10.122 (PA11)
- net USB_DP is gone; now on net OTG_FS_DP: U10.123 (PA12)
- net GND: now also C3.1, LC10.3
- net VCC: now also LC10.1
- net at U1.3 (BYP): now also C3.2
- net I2C2_VCC: no longer names the net of C51.1
- net I2C2_VCC: now also LC10.2
- no-connect marks 71 -> 79
Other:
- moved on the sheet: C2, C4, U1, U3
